File: smart_alarm_V0.1/FP6291.kicad_sch (KiCad schematic)
At the start: 11 parts, among them IC301 FP6291

Commit message: Footprint rearrange
Parts:
- C302, C303: value 20uF -> 22uF
- D301: value D_Shockley -> B340A
- L301: footprint Inductor_SMD:L_Coilcraft_XAL5030-XXX -> Inductor_SMD:L_Taiyo-Yuden_MD-5050
Changed lines of the file:
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@@
       (effects (font (size 1.27 1.27)) (justify left))
     )
-    (property "Value" "20uF" (at 93.98 118.11 0)
+    (property "Value" "22uF" (at 93.98 118.11 0)
       (effects (font (size 1.27 1.27)) (justify left))
     )
@@
       (effects (font (size 1.27 1.27)) (justify left))
     )
-    (property "Value" "20uF" (at 168.91 104.14 0)
+    (property "Value" "22uF" (at 168.91 104.14 0)
       (effects (font (size 1.27 1.27)) (justify left))
     )
@@
       (effects (font (size 1.27 1.27)))
     )
-    (property "Value" "D_Shockley" (at 138.43 90.17 0)
+    (property "Value" "B340A" (at 138.43 90.17 0)
       (effects (font (size 1.27 1.27)))
     )
@@
       (effects (font (size 1.27 1.27)))
     )
-    (property "Footprint" "Inductor_SMD:L_Coilcraft_XAL5030-XXX" (at 113.03 107.95 0)
-      (effects (font (size 1.27 1.27)) hide)
-    )
+    (property "Footprint" "Inductor_SMD:L_Taiyo-Yuden_MD-5050" (at 113.03 107.95 0)
+      (effects (font (size 1.27 1.27)) hide)
+    )
