File: smart_alarm_V0.1/TP4056.kicad_sch (KiCad schematic)
At the start: 16 parts, among them IC201 DW01+G, J201 LI-ION BATTARY, Q201 FS8205A, U201 TP4056

Commit message: Footprint rearrange
Parts:
- C203: value C_Polarized_Small -> 100nF; footprint Capacitor_SMD:C_0603_1608Metric -> Capacitor_SMD:C_0805_2012Metric
- R205: value 100E -> 470E; footprint Resistor_SMD:R_0603_1608Metric -> Resistor_SMD:R_0805_2012Metric
- R206: value R -> 2K
Changed lines of the file:
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@@
       (effects (font (size 1.27 1.27)))
     )
-    (property "Value" "100E" (at 185.42 84.6836 90)
-      (effects (font (size 1.27 1.27)))
-    )
-    (property "Footprint" "Resistor_SMD:R_0603_1608Metric" (at 185.42 85.852 90)
+    (property "Value" "470E" (at 185.42 84.6836 90)
+      (effects (font (size 1.27 1.27)))
+    )
+    (property "Footprint" "Resistor_SMD:R_0805_2012Metric" (at 185.42 85.852 90)
       (effects (font (size 1.27 1.27)) hide)
     )
@@
       (effects (font (size 1.27 1.27)) (justify left))
     )
-    (property "Value" "R" (at 259.588 112.903 0)
+    (property "Value" "2K" (at 259.588 112.903 0)
       (effects (font (size 1.27 1.27)) (justify left))
     )
@@
       (effects (font (size 1.27 1.27)) (justify left))
     )
-    (property "Value" "C_Polarized_Small" (at 181.61 99.06 0)
-      (effects (font (size 1.27 1.27)) (justify left))
-    )
-    (property "Footprint" "Capacitor_SMD:C_0603_1608Metric" (at 193.04 96.52 0)
-      (effects (font (size 1.27 1.27)) hide)
-    )
+    (property "Value" "100nF" (at 194.31 99.06 0)
+      (effects (font (size 1.27 1.27)) (justify left))
+    )
+    (property "Footprint" "Capacitor_SMD:C_0805_2012Metric" (at 193.04 96.52 0)
+      (effects (font (size 1.27 1.27)) hide)
+    )
