File: smart_alarm_V0.1/smart_alarm_V0.1.kicad_pcb (KiCad board)
At the start: 4 copper layers, 60 x 60 mm, 71 parts, among them IC201 DW01+G, IC301 FP6291, IC401 ESP32-C3-WROOM-02-H4, J1 USB_C_Receptacle_PowerOnly_6P, J201 LI-ION BATTARY, J401 JTAG, J403 PROG, Q101 DMG2301L, Q201 FS8205A, SW101 Panic switch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

Commit message: Verify footprint
Parts:
- added G***: LOGO, Custom:Webyfy_Logo_2, F.Cu at (134.4, 51.7)
- SW101: footprint Button_Switch_THT:SW_Push_2P2T_Toggle_CK_PVA2OAH5xxxxxxV2 -> Webyfy:XKB7070Z92
- moved SW101 1.03 mm to (116.9, 67.6), turned to 90 degrees
Routing:
- net /ESP32-C3-WROOM/IO0: track 29.3 -> 28.3 mm
Other:
- board text added: "16-11-2023"
- board text added: "VIN"
- board text added: "VOUT"

Commit message: Footprint rearrange
Parts:
- C203: value C_Polarized_Small -> 100nF; footprint Capacitor_SMD:C_0603_1608Metric -> Capacitor_SMD:C_0805_2012Metric
- C302, C303: value 20uF -> 22uF
- D101: value D_Schottky -> B340
- D301: value D_Shockley -> B340A
- L301: footprint Inductor_SMD:L_Coilcraft_XAL5030-XXX -> Inductor_SMD:L_Taiyo-Yuden_MD-5050
- R101, R102: footprint Resistor_SMD:R_0603_1608Metric -> Resistor_SMD:R_0805_2012Metric
- R205: value 100E -> 470E; footprint Resistor_SMD:R_0603_1608Metric -> Resistor_SMD:R_0805_2012Metric
- R206: value R -> 2K
- moved L301 0.79 mm to (108.5, 69.8)
- moved R101 0.25 mm to (98.8, 72.0)
- moved R102 0.18 mm to (98.8, 70.0)
