File: smart_alarm_V0.1/smart_alarm_V0.1.kicad_sch (KiCad schematic)
At the start: 21 parts, among them J1 USB_C_Receptacle_PowerOnly_6P, Q101 DMG2301L, SW101 Panic switch, SW102 SW_Push, SW103 SW_SPDT

Commit message: Verify footprint
Parts:
- SW101: footprint Button_Switch_THT:SW_Push_2P2T_Toggle_CK_PVA2OAH5xxxxxxV2 -> Webyfy:XKB7070Z92
Changed lines of the file:
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@@
         )
       )
-      (project "power_board_V0.1"
+      (project "smart_alarm_V0.1"
         (path "/6d660399-1d4e-4a8e-97d4-7c2e99e4e5f9/7b458d45-16d8-4976-9083-1e741c84407a"
           (reference "#PWR0406") (unit 1)
@@
     (pin "1")
     (instances
-      (project "power_board_V0.1"
+      (project "smart_alarm_V0.1"
         (path "/6d660399-1d4e-4a8e-97d4-7c2e99e4e5f9/79109c2d-627b-48bd-bc37-0cbd7697e7aa"
           (reference "#PWR0502") (unit 1)
@@
     (pin "2")
     (instances
-      (project "power_board_V0.1"
+      (project "smart_alarm_V0.1"
         (path "/6d660399-1d4e-4a8e-97d4-7c2e99e4e5f9"
           (reference "C101") (unit 1)
@@
     (pin "2")
     (instances
-      (project "power_board_V0.1"
+      (project "smart_alarm_V0.1"
         (path "/6d660399-1d4e-4a8e-97d4-7c2e99e4e5f9/2f5e3b04-97db-4d8f-b6be-02d8e803125e"
           (reference "D202") (unit 1)
@@
     (pin "3")
     (instances
-      (project "power_board_V0.1"
+      (project "smart_alarm_V0.1"
         (path "/6d660399-1d4e-4a8e-97d4-7c2e99e4e5f9"
           (reference "Q101") (unit 1)
@@
     (pin "2")
     (instances
-      (project "power_board_V0.1"
+      (project "smart_alarm_V0.1"
         (path "/6d660399-1d4e-4a8e-97d4-7c2e99e4e5f9"
           (reference "R102") (unit 1)
@@
     (pin "1")
     (instances
-      (project "power_board_V0.1"
+      (project "smart_alarm_V0.1"
         (path "/6d660399-1d4e-4a8e-97d4-7c2e99e4e5f9"
           (reference "#PWR0106") (unit 1)
@@
       (effects (font (size 1.27 1.27)) (justify left))
     )
-    (property "Value" "VBAT" (at 147.32 62.23 0)
+    (property "Value" "VBAT" (at 147.32 72.39 0)
       (effects (font (size 1.27 1.27)) (justify left))
     )
@@
     (pin "1")
     (instances
-      (project "power_board_V0.1"
+      (project "smart_alarm_V0.1"
         (path "/6d660399-1d4e-4a8e-97d4-7c2e99e4e5f9"
           (reference "TP2") (unit 1)
@@
     (pin "2")
     (instances
-      (project "power_board_V0.1"
+      (project "smart_alarm_V0.1"
         (path "/6d660399-1d4e-4a8e-97d4-7c2e99e4e5f9"
           (reference "R101") (unit 1)
@@
     (pin "1")
     (instances
-      (project "power_board_V0.1"
+      (project "smart_alarm_V0.1"
         (path "/6d660399-1d4e-4a8e-97d4-7c2e99e4e5f9/79109c2d-627b-48bd-bc37-0cbd7697e7aa"
           (reference "#PWR0502") (unit 1)
@@
     (pin "2")
     (instances
-      (project "power_board_V0.1"
+      (project "smart_alarm_V0.1"
         (path "/6d660399-1d4e-4a8e-97d4-7c2e99e4e5f9"
           (reference "R105") (unit 1)
@@
     (pin "1")
     (instances
-      (project "power_board_V0.1"
+      (project "smart_alarm_V0.1"
         (path "/6d660399-1d4e-4a8e-97d4-7c2e99e4e5f9"
           (reference "TP6") (unit 1)
@@
     (pin "2")
     (instances
-      (project "power_board_V0.1"
+      (project "smart_alarm_V0.1"
         (path "/6d660399-1d4e-4a8e-97d4-7c2e99e4e5f9"
           (reference "R104") (unit 1)
@@
         )
       )
-      (project "power_board_V0.1"
+      (project "smart_alarm_V0.1"
         (path "/6d660399-1d4e-4a8e-97d4-7c2e99e4e5f9/7b458d45-16d8-4976-9083-1e741c84407a"
           (reference "#PWR0406") (unit 1)
@@
     (pin "1")
     (instances
-      (project "power_board_V0.1"
+      (project "smart_alarm_V0.1"
         (path "/6d660399-1d4e-4a8e-97d4-7c2e99e4e5f9"
           (reference "#PWR0112") (unit 1)
@@
     (pin "1")
     (instances
-      (project "power_board_V0.1"
+      (project "smart_alarm_V0.1"
         (path "/6d660399-1d4e-4a8e-97d4-7c2e99e4e5f9"
           (reference "#PWR0107") (unit 1)
@@
     (pin "S1")
     (instances
-      (project "power_board_V0.1"
+      (project "smart_alarm_V0.1"
         (path "/6d660399-1d4e-4a8e-97d4-7c2e99e4e5f9"
           (reference "J1") (unit 1)
@@
     (pin "1")
     (instances
-      (project "power_board_V0.1"
+      (project "smart_alarm_V0.1"
         (path "/6d660399-1d4e-4a8e-97d4-7c2e99e4e5f9"
           (reference "TP8") (unit 1)
@@
     (pin "1")
     (instances
-      (project "power_board_V0.1"
+      (project "smart_alarm_V0.1"
         (path "/6d660399-1d4e-4a8e-97d4-7c2e99e4e5f9/79109c2d-627b-48bd-bc37-0cbd7697e7aa"
           (reference "#PWR0502") (unit 1)
@@
     (pin "3")
     (instances
-      (project "power_board_V0.1"
+      (project "smart_alarm_V0.1"
         (path "/6d660399-1d4e-4a8e-97d4-7c2e99e4e5f9"
           (reference "SW103") (unit 1)
@@
         )
       )
-      (project "power_board_V0.1"
+      (project "smart_alarm_V0.1"
         (path "/6d660399-1d4e-4a8e-97d4-7c2e99e4e5f9/7b458d45-16d8-4976-9083-1e741c84407a"
           (reference "#PWR0406") (unit 1)
@@
     (pin "2")
     (instances
-      (project "power_board_V0.1"
+      (project "smart_alarm_V0.1"
         (path "/6d660399-1d4e-4a8e-97d4-7c2e99e4e5f9"
           (reference "R106") (unit 1)
@@
     (pin "2")
     (instances
-      (project "power_board_V0.1"
+      (project "smart_alarm_V0.1"
         (path "/6d660399-1d4e-4a8e-97d4-7c2e99e4e5f9"
           (reference "R103") (unit 1)
@@
     (pin "1")
     (instances
-      (project "power_board_V0.1"
+      (project "smart_alarm_V0.1"
         (path "/6d660399-1d4e-4a8e-97d4-7c2e99e4e5f9"
           (reference "TP7") (unit 1)
@@
     (pin "1")
     (instances
-      (project "power_board_V0.1"
+      (project "smart_alarm_V0.1"
         (path "/6d660399-1d4e-4a8e-97d4-7c2e99e4e5f9"
           (reference "#PWR0109") (unit 1)
@@
     (pin "2")
     (instances
-      (project "power_board_V0.1"
+      (project "smart_alarm_V0.1"
         (path "/6d660399-1d4e-4a8e-97d4-7c2e99e4e5f9"
           (reference "D101") (unit 1)
@@
     (pin "2")
     (instances
-      (project "power_board_V0.1"
+      (project "smart_alarm_V0.1"
         (path "/6d660399-1d4e-4a8e-97d4-7c2e99e4e5f9"
           (reference "FB101") (unit 1)
@@
     (pin "2")
     (instances
-      (project "power_board_V0.1"
+      (project "smart_alarm_V0.1"
         (path "/6d660399-1d4e-4a8e-97d4-7c2e99e4e5f9"
           (reference "FB102") (unit 1)
@@
     (pin "1")
     (instances
-      (project "power_board_V0.1"
+      (project "smart_alarm_V0.1"
         (path "/6d660399-1d4e-4a8e-97d4-7c2e99e4e5f9/79109c2d-627b-48bd-bc37-0cbd7697e7aa"
           (reference "#PWR0502") (unit 1)
@@
       (effects (font (size 1.27 1.27)))
     )
-    (property "Footprint" "Button_Switch_THT:SW_Push_2P2T_Toggle_CK_PVA2OAH5xxxxxxV2" (at 210.82 101.6 0)
+    (property "Footprint" "Webyfy:XKB7070Z92" (at 210.82 101.6 0)
       (effects (font (size 1.27 1.27)) hide)
     )
@@
     (pin "6")
     (instances
-      (project "power_board_V0.1"
+      (project "smart_alarm_V0.1"
         (path "/6d660399-1d4e-4a8e-97d4-7c2e99e4e5f9"
           (reference "SW101") (unit 1)
@@
     (pin "1")
     (instances
-      (project "power_board_V0.1"
+      (project "smart_alarm_V0.1"
         (path "/6d660399-1d4e-4a8e-97d4-7c2e99e4e5f9/79109c2d-627b-48bd-bc37-0cbd7697e7aa"
           (reference "#PWR0502") (unit 1)
@@
     (pin "2")
     (instances
-      (project "power_board_V0.1"
+      (project "smart_alarm_V0.1"
         (path "/6d660399-1d4e-4a8e-97d4-7c2e99e4e5f9"
           (reference "SW102") (unit 1)
@@
     (pin "1")
     (instances
-      (project "power_board_V0.1"
+      (project "smart_alarm_V0.1"
         (path "/6d660399-1d4e-4a8e-97d4-7c2e99e4e5f9"
           (reference "TP3") (unit 1)
@@
         (path "/c6785104-e587-4344-83f1-abbec1041e77/00000000-0000-0000-0000-000061c99eb6" (page "6"))
       )
-      (project "power_board_V0.1"
+      (project "smart_alarm_V0.1"
         (path "/6d660399-1d4e-4a8e-97d4-7c2e99e4e5f9" (page "2"))
       )
@@
     )
     (instances
-      (project "power_board_V0.1"
+      (project "smart_alarm_V0.1"
         (path "/6d660399-1d4e-4a8e-97d4-7c2e99e4e5f9" (page "5"))
       )
@@
     )
     (instances
-      (project "power_board_V0.1"
+      (project "smart_alarm_V0.1"
         (path "/6d660399-1d4e-4a8e-97d4-7c2e99e4e5f9" (page "4"))
       )
@@
         (path "/c6785104-e587-4344-83f1-abbec1041e77/00000000-0000-0000-0000-000061c99eb6" (page "7"))
       )
-      (project "power_board_V0.1"
+      (project "smart_alarm_V0.1"
         (path "/6d660399-1d4e-4a8e-97d4-7c2e99e4e5f9" (page "3"))
       )

Commit message: Footprint rearrange
Parts:
- D101: value D_Schottky -> B340
- R101, R102: footprint Resistor_SMD:R_0603_1608Metric -> Resistor_SMD:R_0805_2012Metric
Changed lines of the file:
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@@
       (effects (font (size 1.27 1.27)) (justify left))
     )
-    (property "Footprint" "Resistor_SMD:R_0603_1608Metric" (at 73.152 132.08 90)
+    (property "Footprint" "Resistor_SMD:R_0805_2012Metric" (at 73.152 132.08 90)
       (effects (font (size 1.27 1.27)) hide)
     )
@@
       (effects (font (size 1.27 1.27)) (justify left))
     )
-    (property "Footprint" "Resistor_SMD:R_0603_1608Metric" (at 73.152 114.3 90)
+    (property "Footprint" "Resistor_SMD:R_0805_2012Metric" (at 73.152 114.3 90)
       (effects (font (size 1.27 1.27)) hide)
     )
@@
       (effects (font (size 1.27 1.27)))
     )
-    (property "Value" "D_Schottky" (at 176.53 48.8696 0)
-      (effects (font (size 1.27 1.27)))
-    )
+    (property "Value" "B340" (at 176.53 48.8696 0)
+      (effects (font (size 1.27 1.27)))
+    )
